Commit message: Kinematics node working as it should

File: src/snakebot_description/urdf/macros.xacro (robot description, xacro)
@@ -83,5 +83,5 @@
 	</transmission>
 	</macro>
-	<macro name="body_upTo9" params="num nextNum">
+	<macro name="body_upTo3" params="num nextNum">
 	<link name="body_0${num}">
 		<collision>
@@ -142,5 +142,5 @@
 	</transmission>
 	</macro>
-		<macro name="body_9" params="num nextNum">
+		<macro name="body_3" params="num nextNum">
 	<link name="body_0${num}">
 		<collision>
@@ -201,5 +201,5 @@
 	</transmission>
 	</macro>
-	<macro name="body_last_upTo9" params="num">
+	<macro name="body_last_upTo3" params="num">
 	<link name="body_0${num}">
 		<collision>
@@ -242,5 +242,5 @@
 	</gazebo>
 	</macro>
-	<macro name="body_above9" params="num nextNum">
+	<macro name="body_above3" params="num nextNum">
 	<link name="body_${num}">
 		<collision>
@@ -301,5 +301,5 @@
 	</transmission>
 	</macro>
-	<macro name="body_last_above9" params="num">
+	<macro name="body_last_above3" params="num">
 	<link name="body_${num}">
 		<collision>

File: src/snakebot_description/urdf/snakebot.xacro (robot description, xacro)
@@ -28,17 +28,11 @@
 	</joint>
 	<body_first num="1" nextNum="2"/>
-	<body_upTo9 num="2" nextNum="3"/>
-	<body_upTo9 num="3" nextNum="4"/>
-	<body_upTo9 num="4" nextNum="5"/>
-	<body_upTo9 num="5" nextNum="6"/>
-	<body_upTo9 num="6" nextNum="7"/>
-	<body_upTo9 num="7" nextNum="8"/>
-	<body_upTo9 num="8" nextNum="9"/>
-	<body_9 num="9" nextNum="10"/>
-	<body_above9 num="10" nextNum="11"/>
-	<body_last_above9 num="11"/>
+	<body_upTo3 num="2" nextNum="3"/>
+	<body_3 num="3" nextNum="4"/>
+	<body_above3 num="4" nextNum="5"/>
+	<body_last_above3 num="5"/>
   <joint name="camera_joint" type="fixed">
     <origin xyz="${camera_link+chassisLength} 0 ${0.5*camera_link}" rpy="0 0 0"/>
-    <parent link="body_11"/>
+    <parent link="body_5"/>
     <child link="camera_link"/>
   </joint>

Commit message: Changed snake config back to 11 links

File: src/snakebot_description/urdf/macros.xacro (robot description, xacro)
@@ -83,5 +83,5 @@
 	</transmission>
 	</macro>
-	<macro name="body_upTo3" params="num nextNum">
+	<macro name="body_upTo9" params="num nextNum">
 	<link name="body_0${num}">
 		<collision>
@@ -142,5 +142,5 @@
 	</transmission>
 	</macro>
-		<macro name="body_3" params="num nextNum">
+		<macro name="body_9" params="num nextNum">
 	<link name="body_0${num}">
 		<collision>
@@ -201,5 +201,5 @@
 	</transmission>
 	</macro>
-	<macro name="body_last_upTo3" params="num">
+	<macro name="body_last_upTo9" params="num">
 	<link name="body_0${num}">
 		<collision>
@@ -242,5 +242,5 @@
 	</gazebo>
 	</macro>
-	<macro name="body_above3" params="num nextNum">
+	<macro name="body_above9" params="num nextNum">
 	<link name="body_${num}">
 		<collision>
@@ -301,5 +301,5 @@
 	</transmission>
 	</macro>
-	<macro name="body_last_above3" params="num">
+	<macro name="body_last_above9" params="num">
 	<link name="body_${num}">
 		<collision>

File: src/snakebot_description/urdf/snakebot.xacro (robot description, xacro)
@@ -28,11 +28,17 @@
 	</joint>
 	<body_first num="1" nextNum="2"/>
-	<body_upTo3 num="2" nextNum="3"/>
-	<body_3 num="3" nextNum="4"/>
-	<body_above3 num="4" nextNum="5"/>
-	<body_last_above3 num="5"/>
+    <body_upTo9 num="2" nextNum="3"/>
+    <body_upTo9 num="3" nextNum="4"/>
+    <body_upTo9 num="4" nextNum="5"/>
+    <body_upTo9 num="5" nextNum="6"/>
+    <body_upTo9 num="6" nextNum="7"/>
+    <body_upTo9 num="7" nextNum="8"/>
+    <body_upTo9 num="8" nextNum="9"/>
+    <body_9 num="9" nextNum="10"/>
+    <body_above9 num="10" nextNum="11"/>
+    <body_last_above9 num="11"/>
   <joint name="camera_joint" type="fixed">
     <origin xyz="${camera_link+chassisLength} 0 ${0.5*camera_link}" rpy="0 0 0"/>
-    <parent link="body_5"/>
+    <parent link="body_11"/>
     <child link="camera_link"/>
   </joint>
