Commit message: Commit before Easter. POAL working with reduced resolution on force data.

File: src/snakebot_description/urdf/snakebot.xacro (robot description, xacro)
@@ -6,10 +6,10 @@
   <xacro:property name="axel_offset" value="0.05" /> <!-- Space btw top of beam and the each joint -->
 	<xacro:property name="PI" value="3.1415926535897931"/>
-	<xacro:property name="chassisHeight" value="0.1"/>
-	<xacro:property name="chassisLength" value="0.2"/>
-	<xacro:property name="chassisWidth" value="0.1"/>
-	<xacro:property name="chassisMass" value="1"/>
-	<xacro:property name="jointOffset" value="0.03"/>
-	<xacro:property name="casterRadius" value="0.05"/>
+	<xacro:property name="chassisHeight" value="0.1"/><!--Simulation:0.1 Real robot: 0.07-->
+	<xacro:property name="chassisLength" value="0.2"/><!--Simulation: 0.2 Real robot: 0.0885-->
+	<xacro:property name="chassisWidth" value="0.1"/><!--Simulation: 0.1 Real robot: 0.07-->
+	<xacro:property name="chassisMass" value="1"/><!--1-->
+	<xacro:property name="jointOffset" value="0.03"/> <!--Simulation: 0.03 Real robot: 0.01-->
+	<xacro:property name="casterRadius" value="0.05"/><!--0.05-->
 	<xacro:property name="casterMass" value="5"/>
 	<xacro:property name="wheelWidth" value="0.05"/>
@@ -27,5 +27,5 @@
 		<child link="body_01"/>
 	</joint>
-	<body_first num="1" nextNum="2"/>
+  <body_first num="1" nextNum="2"/>
     <body_upTo9 num="2" nextNum="3"/>
     <body_upTo9 num="3" nextNum="4"/>
@@ -37,8 +37,11 @@
     <body_9 num="9" nextNum="10"/>
     <body_above9 num="10" nextNum="11"/>
-    <body_last_above9 num="11"/>
+    <body_above9 num="11" nextNum="12"/>
+    <body_above9 num="12" nextNum="13"/>
+    <body_above9 num="13" nextNum="14"/>
+    <body_last_above9 num="14"/>
   <joint name="camera_joint" type="fixed">
     <origin xyz="${camera_link+chassisLength} 0 ${0.5*camera_link}" rpy="0 0 0"/>
-    <parent link="body_11"/>
+    <parent link="body_14"/>
     <child link="camera_link"/>
   </joint>

Commit message: Working POAL with angle controller. Push points farthest towards the head are being applied. RViz shows nearest joint as push point. Forces are not displayed accurately

File: src/snakebot_description/urdf/snakebot.xacro (robot description, xacro)
@@ -6,9 +6,9 @@
   <xacro:property name="axel_offset" value="0.05" /> <!-- Space btw top of beam and the each joint -->
 	<xacro:property name="PI" value="3.1415926535897931"/>
-	<xacro:property name="chassisHeight" value="0.1"/><!--Simulation:0.1 Real robot: 0.07-->
-	<xacro:property name="chassisLength" value="0.2"/><!--Simulation: 0.2 Real robot: 0.0885-->
-	<xacro:property name="chassisWidth" value="0.1"/><!--Simulation: 0.1 Real robot: 0.07-->
+	<xacro:property name="chassisHeight" value="0.07"/><!--Simulation:0.1 Real robot: 0.07-->
+	<xacro:property name="chassisLength" value="0.0885"/><!--Simulation: 0.2 Real robot: 0.0885-->
+	<xacro:property name="chassisWidth" value="0.07"/><!--Simulation: 0.1 Real robot: 0.07-->
 	<xacro:property name="chassisMass" value="1"/><!--1-->
-	<xacro:property name="jointOffset" value="0.03"/> <!--Simulation: 0.03 Real robot: 0.01-->
+	<xacro:property name="jointOffset" value="0.01"/> <!--Simulation: 0.03 Real robot: 0.01-->
 	<xacro:property name="casterRadius" value="0.05"/><!--0.05-->
 	<xacro:property name="casterMass" value="5"/>
